Commit message: updated joint limits

File: cr5_moveit/config/gazebo_cr5_robot.urdf (robot description, URDF)
Before this commit: robot cr5_robot, 8 links, 7 joints
Joints:
- joint joint2: limit lower=-1.74533 upper=1.74533 effort=0 velocity=0 -> lower=0.174533 upper=1.74533 effort=0 velocity=0
- joint joint3: limit lower=0 upper=2.79253 effort=0 velocity=0 -> lower=0.174533 upper=2.79253 effort=0 velocity=0

File: dobot_description/urdf/cr5_robot.urdf (robot description, URDF)
Before this commit: robot cr5_robot, 8 links, 7 joints
Joints:
- joint joint2: limit lower=-1.74533 upper=1.74533 effort=0 velocity=0 -> lower=0.174533 upper=1.74533 effort=0 velocity=0
- joint joint3: limit lower=0 upper=2.79253 effort=0 velocity=0 -> lower=0.174533 upper=2.79253 effort=0 velocity=0

Commit message: changes to joint limit of joint 2 based on additional testing

File: cr5_moveit/config/gazebo_cr5_robot.urdf (robot description, URDF)
Before this commit: robot cr5_robot, 8 links, 7 joints
Joints:
- joint joint2: limit lower=0.174533 upper=1.74533 effort=0 velocity=0 -> lower=-0.785398 upper=1.74533 effort=0 velocity=0

File: dobot_description/urdf/cr5_robot.urdf (robot description, URDF)
Before this commit: robot cr5_robot, 8 links, 7 joints
Joints:
- joint joint2: limit lower=0.174533 upper=1.74533 effort=0 velocity=0 -> lower=-0.785398 upper=1.74533 effort=0 velocity=0
