Commit message: parameter adjustments

File: dobot_description/urdf/cr5_robot.urdf (robot description, URDF)
Before this commit: robot cr5_robot, 8 links, 7 joints
Joints:
- joint joint2: limit lower=-0.785398 upper=1.74533 effort=0 velocity=0 -> lower=-1.74533 upper=0.785398 effort=0 velocity=0
- joint joint3: limit lower=0.174533 upper=2.79253 effort=0 velocity=0 -> lower=-2.79253 upper=-0.174533 effort=0 velocity=0
